File: hardware/schem.sch (EAGLE design)
At the start: 5 parts, among them U1 ATTINY85-20P

Commit message: Updated schematic for board
Parts:
- added C3: 3.3n, SparkFun-Capacitors:CAPEZ
- added C4: 47n, SparkFun-Capacitors:CAPEZ
- added C5: 100u, resistor:CPOL-USE2-5
- added ISP1: AVRISP-6, adafruit:AVRISP-6
- added Q1: IRF540, transistor-fet:IRF540
- added R3: 56, SparkFun-Passives:RESISTORAXIAL-0.3
- C1, C2: value (none) -> 1uF; device SparkFun-Capacitors:CAPPTH2 -> capacitor-wima:C2.5/6
- R1, R2: value (none) -> 10k; device SparkFun-Passives:RESISTOREZ -> SparkFun-Passives:RESISTORAXIAL-0.3
Connections:
- net OUT renamed TH
- removed net N$10: C1.1, R1.2, R2.1
- removed net N$3: R1.1, U1.PB0
- removed net SW-IN: U1.PB1
- removed net THR-IN: U1.PB2
- new net BR-IN: C4.1, U1.PB4
- new net BR-SW: Q1.D
- new net BRK-AN: C1.1, R1.2
- new net MISO: ISP1.MISO, R1.1, U1.PB1
- new net MOSI: ISP1.MOSI, R2.1, U1.PB0
- new net N$1: R3.1, U1.PB3
- new net N$2: Q1.G, R3.2
- new net RST: ISP1.RST, U1.NRES/PB5
- new net TH-IN: ISP1.SCK, U1.PB2
- net +5V: now also C3.1, C5.+, ISP1.VCC
- net GND: now also C3.2, C4.2, C5.-, ISP1.GND, Q1.S; no longer C1.2
Other:
- moved on the sheet: C1, C2, R1, R2, U1
